File: schematic/pslab-mini.kicad_pcb (KiCad board)
At the start: 4 copper layers, 85 x 56 mm, 150 parts, among them J1 USB_C_Receptacle_USB2.0_16P, J2 Battery_Cell, J3 Conn_Coaxial, J4 Conn_Coaxial, J6 Conn_01x16_Socket, J7 Conn_02x03_Top_Bottom, J8 Conn_02x17_Odd_Even, Q1 MMBT3904, Q2 MMBT3906, SW1 Power, SW2 Reset, U1 MT1470, U10 TL082, U11 ESP32-C3, U2 AP3015A, U3 IP5189T, U4 SP0503BAHT, U5 AMS1117-3.3, U6 STM32H563RIT6, U7 TL082, U8 MCP6S21, U9 MCP6S21, X1 32kHz768, Y1 Crystal_25MHz, Y2 Crystal_40Mhz

Commit message: pcb1
Parts:
- moved J2 41.9 mm to (132.6, 102.0)
- moved J6 10.0 mm to (87.5, 106.0)
Changed lines of the file:
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@@
 	(footprint "Connector_PinSocket_2.54mm:PinSocket_1x16_P2.54mm_Vertical"
 		(layer "F.Cu")
-		(at 97.5 105.975 90)
+		(at 87.5 105.975 90)
 		(descr "Through hole straight socket strip, 1x16, 2.54mm pitch, single row (from Kicad 4.0.7), script generated")
 		(tags "Through hole socket strip THT 1x16 2.54mm single row")
@@
 	(footprint "pslab-mini:2.0mm_connector_edge"
 		(layer "F.Cu")
-		(at 90.75 99.6 180)
+		(at 132.55 102 180)
 		(property "Reference" "J2"
 			(at -5.1 0.8 0)
