File: schematic/pslab-mini.kicad_pcb (KiCad board)
At the start: 4 copper layers, 85 x 56 mm, 145 parts, among them J1 USB_C_Receptacle_USB2.0_16P, J2 Battery_Cell, J3 Conn_Coaxial, J4 Conn_Coaxial, J5 Conn_02x18_Odd_Even, J6 Conn_01x15_Socket, J7 Conn_02x03_Top_Bottom, Q1 MMBT3904, Q2 MMBT3906, SW1 Reset, SW2 Power, U1 MT1470, U10 TL082, U11 ESP32-C3, U2 AP3015A, U3 IP5189T, U4 SP0503BAHT, U5 AMS1117-3.3, U6 STM32H563RIT6, U7 TL082, U8 MCP6S21, U9 MCP6S21, X1 32kHz768, Y1 Crystal_25MHz, Y2 Crystal_40Mhz

Commit message: routing
Parts:
- moved TP2 5.53 mm to (154.1, 96.5)
- moved TP6 4.35 mm to (154.1, 101.1)
- moved U4 1.35 mm to (150.5, 97.9), turned to 90 degrees
- moved C30 1.25 mm to (117.9, 70.3), turned to -90 degrees
- moved R1 1.12 mm to (138.6, 91.6)
- moved TP3 0.88 mm to (125.5, 86.2)
- moved R29 0.80 mm to (138.5, 76.2)
- moved Y1 0.69 mm to (118.5, 75.0)
- moved TP5 0.61 mm to (122.7, 83.0)
- moved TP4 0.58 mm to (154.1, 98.8)
- moved R13 0.55 mm to (120.5, 72.0)
- moved C16 0.44 mm to (122.5, 73.8)
- moved C31 0.39 mm to (120.5, 70.1)
- moved C28 0.38 mm to (98.2, 66.0)
- moved C14 0.38 mm to (122.5, 75.7)
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Connections:
- J5 pad 1: Net-(J5-Pin_1) -> GND
- J5 pad 11: Net-(J5-Pin_1) -> GND
- J5 pad 13: Net-(J5-Pin_1) -> GND
- J5 pad 15: Net-(J5-Pin_1) -> GND
- J5 pad 17: Net-(J5-Pin_1) -> GND
- J5 pad 3: Net-(J5-Pin_1) -> GND
- J5 pad 5: Net-(J5-Pin_1) -> GND
- J5 pad 7: Net-(J5-Pin_1) -> GND
- J5 pad 9: Net-(J5-Pin_1) -> GND
Routing:
- net +3V3: track 0.00 -> 234.4 mm, vias 0 -> 11
- net VDDA: track 0.00 -> 135.6 mm, vias 0 -> 11
- net GND: track 0.00 -> 114.8 mm, vias 0 -> 114
- net +5V: track 0.00 -> 98.3 mm, vias 0 -> 4
- net /D-: track 0.00 -> 72.4 mm, vias 0 -> 2
- net /D+: track 0.00 -> 69.8 mm, vias 0 -> 2
- net /UART6_TX: track 0.00 -> 41.2 mm, vias 0 -> 1
- net /UART6_RX: track 0.00 -> 39.7 mm, vias 0 -> 1
- net /NRST: track 0.00 -> 38.7 mm
- net /VINPUT: track 0.00 -> 34.5 mm, vias 0 -> 3
- net +6V: track 0.00 -> 34.4 mm, vias 0 -> 3
- net /I2C1_SDA: track 0.00 -> 34.2 mm, vias 0 -> 2
- net /I2C1_SCL: track 0.00 -> 32.7 mm, vias 0 -> 2
- net /SPI.CS: track 0.00 -> 31.4 mm
- net -6V: track 0.00 -> 30.7 mm, vias 0 -> 2
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- added copper zone on F.Cu, net GND
- added copper zone on In1.Cu, net GND

Commit message: MC34063ADR
Parts:
- removed C1, C8, C9: 22uF, Capacitor_SMD:C_0805_2012Metric
- removed C4: 1uF, Capacitor_SMD:C_0603_1608Metric
- removed C6: 12pF, Capacitor_SMD:C_0603_1608Metric
- removed D4: 6.8V, Diode_SMD:D_SOD-123
- removed D5: 1N4148W, Diode_SMD:D_SOD-123
- removed L2: 3.3uH, Inductor_SMD:L_0603_1608Metric
- removed Q2: MMBT3906, Package_TO_SOT_SMD:SOT-23
- removed R11: 1k, Resistor_SMD:R_0603_1608Metric
- removed R2: 200k, Resistor_SMD:R_0603_1608Metric
- removed R6: 100k, Resistor_SMD:R_0603_1608Metric
- removed R7: 10k, Resistor_SMD:R_0603_1608Metric
- removed U1: MT1470, Package_TO_SOT_SMD:SOT-23-6
- added C46: 100uF, Capacitor_SMD:C_0603_1608Metric, F.Cu at (116.2, 86.8)
- added C47: 1.5nF, Capacitor_SMD:C_0603_1608Metric, F.Cu at (126.5, 88.6)
- added C48: 1000uF, Capacitor_SMD:C_0603_1608Metric, F.Cu at (131.3, 88.5)
- added C49: 100uF, Capacitor_SMD:C_0603_1608Metric, F.Cu at (130.4, 86.0)
- added D13: 1N5819WS, Diode_SMD:D_SOD-323, F.Cu at (129.2, 88.8)
- added D14: 6.8V, Diode_SMD:D_SOD-123, F.Cu at (128.8, 82.5)
- added D15: 1N4148W, Diode_SMD:D_SOD-123, F.Cu at (125.1, 80.5)
- added L6: 88uH, Inductor_SMD:L_0603_1608Metric, F.Cu at (127.2, 91.5)
- added L7: 1uH, Inductor_SMD:L_0603_1608Metric, F.Cu at (127.2, 86.0)
- added Q3: MMBT3906, Package_TO_SOT_SMD:SOT-23, F.Cu at (123.0, 84.1)
- added R40: 0.24R, Resistor_SMD:R_0603_1608Metric, F.Cu at (116.9, 90.6)
- added R41: 1k, Resistor_SMD:R_0603_1608Metric, F.Cu at (119.3, 85.2)
- added R42: 6.2k, Resistor_SMD:R_0603_1608Metric, F.Cu at (119.0, 83.5)
- added R43: 1k, Resistor_SMD:R_0603_1608Metric, F.Cu at (126.3, 83.5)
- added U12: MC34063ADR, Package_SO:SOIC-8_3.9x4.9mm_P1.27mm, F.Cu at (121.7, 89.1)
- moved TP5 2.08 mm to (121.0, 81.8)
- moved TP3 0.65 mm to (124.9, 85.8)
Routing:
- net Net-(D13-A): track 0.00 -> 13.9 mm
- net Net-(U12-DC): track 0.00 -> 8.63 mm
- net -9V: track 17.5 -> 9.66 mm
- net Net-(D5-K): track 6.60 -> 0.00 mm
- net Net-(D13-K): track 0.00 -> 6.50 mm
- net Net-(U1-SW): track 5.95 -> 0.00 mm
- net Net-(U1-FB): track 5.62 -> 0.00 mm
- net Net-(D15-K): track 0.00 -> 5.45 mm
- net Net-(U12-Vfb): track 0.00 -> 4.16 mm
- net Net-(U1-EN): track 3.84 -> 0.00 mm
- net -6V: track 30.7 -> 33.7 mm, vias 2 -> 3
- net Net-(U12-TC): track 0.00 -> 2.75 mm
- net Net-(D14-A): track 0.00 -> 2.24 mm
- net Net-(U1-BST): track 2.19 -> 0.00 mm
- net Net-(D4-A): track 2.04 -> 0.00 mm
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Other:
- board text removed: "-9V"
