File: schematic/pslab-mini.kicad_sch (KiCad schematic)
At the start: 152 parts, among them J1 USB_C_Receptacle_USB2.0_16P, J2 Battery_Cell, J3 Conn_Coaxial, J4 Conn_Coaxial, J5 Conn_02x13_Odd_Even, J6 Conn_01x16_Socket, J7 Conn_02x03_Top_Bottom, Q1 MMBT3904, Q2 MMBT3906, SW1 Power, SW2 Reset, SW3 Boot, U1 MT1470, U10 TL082, U11 ESP32-C3, U2 AP3015A, U3 IP5189T, U4 SP0503BAHT, U5 AMS1117-3.3, U6 STM32H563RIT6, U7 TL082, U8 MCP6S21, U9 MCP6S21, X1 32kHz768, Y1 Crystal_25MHz, Y2 Crystal_40Mhz

Commit message: Naming reconfiguration and removing the BOOT0 button
Parts:
- removed J5: Conn_02x13_Odd_Even, Connector_PinSocket_2.54mm:PinSocket_2x13_P2.54mm_Vertical, symbol Connector_Generic:Conn_02x13_Odd_Even
- removed R15: 10k, Resistor_SMD:R_0603_1608Metric, symbol Device:R
- removed SW3: Boot, Button_Switch_SMD:SW_Tactile_SPST_NO_Straight_CK_PTS636Sx25SMTRLFS, symbol Switch:SW_Push
- added J8: Conn_02x17_Odd_Even, Connector_PinSocket_2.54mm:PinSocket_2x17_P2.54mm_Vertical, symbol Connector_Generic:Conn_02x17_Odd_Even
- D6: Mfr Number WS2812B-V5 -> WS2812B-B/W; Part Number (LCSC) C2846931 -> C114586
- MH1, MH2, MH3, MH4: footprint MountingHole:MountingHole_3.2mm_M3_Pad -> pslab-mini:MountingHole_2.75mm_Pad
Connections:
- net BOOT0 is gone; now on net GND: U6.60 (BOOT0)
- net PC7 is gone; now on an unnamed net: U6.38 (PC7)
- net CAP: now also J8.14 (Pin_14)
- net CH1: now also J8.2 (Pin_2)
- net CH2: now also J8.4 (Pin_4)
- net FQY: now also J8.16 (Pin_16)
- net GND: now also J8.1 (Pin_1), J8.11 (Pin_11), J8.13 (Pin_13), J8.15 (Pin_15), J8.17 (Pin_17), J8.19 (Pin_19), J8.21 (Pin_21), J8.23 (Pin_23), J8.25 (Pin_25), J8.27 (Pin_27), J8.29 (Pin_29), J8.3 (Pin_3), J8.31 (Pin_31), J8.33 (Pin_33), J8.5 (Pin_5), J8.7 (Pin_7), J8.9 (Pin_9)
- net LA1: now also J8.6 (Pin_6)
- net LA2: now also J8.8 (Pin_8)
- net RES: now also J8.12 (Pin_12)
- net USER_LED: now also U6.57 (PB5); no longer U6.26 (PB0)
- net VOL: now also J8.10 (Pin_10)
- net at R12.2: now also U6.35 (PB14); no longer U6.24 (PC4)
- net GPIO0: now reaches U6.20 (PA4)
- net GPIO0: now also J8.18 (Pin_18)
- net at R13.2: no longer U6.25 (PC5)
- net GPIO7: now reaches U6.40 (PC9)
- net GPIO7: now also J8.32 (Pin_32)
- net KEY: now reaches SW1.2, U3.8 (KEY)
- net PB10 renamed GPIO5
- net GPIO5: now also J8.28 (Pin_28)
- net PB8 renamed GPIO4
- net GPIO4: now also J8.26 (Pin_26)
- net PC8 renamed GPIO6
- net GPIO6: now also J8.30 (Pin_30)
- net SQRT renamed SQR
- net SQR: now also J8.34 (Pin_34)
- new net GPIO1: J8.20 (Pin_20), U6.26 (PB0)
- new net GPIO2: J8.22 (Pin_22), U6.24 (PC4)
- new net GPIO3: J8.24 (Pin_24), U6.25 (PC5)
- no-connect marks 31 -> 27
Other:
- note added: "Analog Input"
- note added: "Digital Input"
- note added: "I2C"
- note added: "Logic Analyser"
- note added: "Multimeter"
- note added: "Oscilloscope"
- note added: "SPI"
- note added: "Square Wave"
- note added: "UART"
- moved on the sheet: D6, J6, R12, R13, R14, SW1

Commit message: Completed layout
Parts:
- J7: footprint TerminalBlock_WAGO:TerminalBlock_WAGO_233-503_2x03_P2.54mm -> pslab-mini:pslab-mini_2x03_P2.54mm

Commit message: sch and pro
Parts:
- D+1: renamed from TP7; value D- -> TP7
- D-1: renamed from TP8; value VINBUS -> TP8
- GND1: renamed from TP9; value GND -> TP9
- VUSBIN1: renamed from TP6; value D+ -> TP6
- renumbered J8 to J5, R14 to R12, R16 to R14, R17 to R15, R18 to R16, R19 to R17, R20 to R18, R21 to R19, R22 to R20, R23 to R21, R24 to R22, R25 to R23, R12 to R24, R26 to R25, R27 to R26, R28 to R27, R29 to R28, R30 to R29, R31 to R30, R32 to R31, R33 to R32, R34 to R33, R35 to R34, R36 to R35, R37 to R36, R38 to R37, R39 to R38, R40 to R39, SW2 to SW1, SW1 to SW2

Commit message: new layout
Parts:
- removed R12, R13: 200, Resistor_SMD:R_0603_1608Metric, symbol Device:R
- added R40, R41: 200, Resistor_SMD:R_0603_1608Metric, symbol Device:R
Connections:
- net CAP: now also J5.22 (Pin_22); no longer J5.14 (Pin_14)
- net CH1: now also J5.34 (Pin_34); no longer J5.2 (Pin_2)
- net CH2: now also J5.32 (Pin_32); no longer J5.4 (Pin_4)
- net CS1: now also U6.16 (PA2); no longer U6.27 (PB1)
- net CS2: now also U6.17 (PA3); no longer U6.28 (PB2)
- net FQY: now also J5.20 (Pin_20), R40.1; no longer J5.16 (Pin_16), R24.1
- net GPIO1: now also J5.16 (Pin_16); no longer J5.20 (Pin_20)
- net GPIO2: now also J5.14 (Pin_14); no longer J5.22 (Pin_22)
- net GPIO3: now also J5.12 (Pin_12); no longer J5.24 (Pin_24)
- net GPIO4: now also J5.10 (Pin_10), U6.2 (PC13); no longer J5.26 (Pin_26), U6.61 (PB8)
- net GPIO5: now also J5.8 (Pin_8); no longer J5.28 (Pin_28)
- net GPIO6: now also J5.6 (Pin_6); no longer J5.30 (Pin_30)
- net GPIO7: now also J5.4 (Pin_4); no longer J5.32 (Pin_32)
- net LA1: now also J5.30 (Pin_30), R41.1; no longer J5.6 (Pin_6)
- net LA2: now also J5.28 (Pin_28), R24.1; no longer J5.8 (Pin_8)
- net RES: now also J5.24 (Pin_24); no longer J5.12 (Pin_12)
- net RGB: now also U6.61 (PB8); no longer U6.2 (PC13)
- net SPI1_MOSI: now also U8.6 (SDI), U9.6 (SDI); no longer R38.1
- net SPI1_SCK: now also U8.7 (SCK), U9.7 (SCK); no longer R37.1
- net SPI2_MOSI: now also R38.1; no longer U8.6 (SDI), U9.6 (SDI)
- net SPI2_SCK: now also R37.1; no longer U8.7 (SCK), U9.7 (SCK)
- net SQR: now also J5.2 (Pin_2); no longer J5.34 (Pin_34)
- net VOL: now also J5.26 (Pin_26); no longer J5.10 (Pin_10)
- net at R24.2: now also U6.28 (PB2); no longer U6.35 (PB14)
- net UART6_TX: now reaches U6.37 (PC6)
- net UART6_TX: now also J6.3 (Pin_3)
- net UART6_RX: now reaches U6.38 (PC7)
- net UART6_RX: now also J6.4 (Pin_4)
- net SPI1_MISO: no longer names the net of U6.22 (PA6)
- net SPI1_MISO: now also R40.2; no longer R39.1
- removed net UART2_RX: J6.4 (Pin_4), U6.17 (PA3)
- removed net UART2_TX: J6.3 (Pin_3), U6.16 (PA2)
- new net: R41.2, U6.27 (PB1)
- new net SPI2_MISO: R39.1, U6.35 (PB14)
Other:
- moved on the sheet: R22, R23

Commit message: new routing
Connections:
- net CH1: now also J5.32 (Pin_32); no longer J5.34 (Pin_34)
- net CH2: now also J5.34 (Pin_34); no longer J5.32 (Pin_32)
- net LA1: now also J5.28 (Pin_28), R24.1; no longer J5.30 (Pin_30), R41.1
- net LA2: now also J5.30 (Pin_30), R41.1; no longer J5.28 (Pin_28), R24.1
