File: schematic/pslab-mini.kicad_sch (KiCad schematic)
At the start: 145 parts, among them J1 USB_C_Receptacle_USB2.0_16P, J2 Battery_Cell, J3 Conn_Coaxial, J4 Conn_Coaxial, J5 Conn_02x18_Odd_Even, J6 Conn_01x15_Socket, J7 Conn_02x03_Top_Bottom, Q1 MMBT3904, Q2 MMBT3906, SW1 Reset, SW2 Power, U1 MT1470, U10 TL082, U11 ESP32-C3, U2 AP3015A, U3 IP5189T, U4 SP0503BAHT, U5 AMS1117-3.3, U6 STM32H563RIT6, U7 TL082, U8 MCP6S21, U9 MCP6S21, X1 32kHz768, Y1 Crystal_25MHz, Y2 Crystal_40Mhz

Commit message: routing
Connections:
- net GND: now also J5.1 (Pin_1), J5.11 (Pin_11), J5.13 (Pin_13), J5.15 (Pin_15), J5.17 (Pin_17), J5.3 (Pin_3), J5.5 (Pin_5), J5.7 (Pin_7), J5.9 (Pin_9)

Commit message: MC34063ADR
Parts:
- removed C1, C8, C9: 22uF, Capacitor_SMD:C_0805_2012Metric, symbol Device:C_Small
- removed C4: 1uF, Capacitor_SMD:C_0603_1608Metric, symbol Device:C_Small
- removed C6: 12pF, Capacitor_SMD:C_0603_1608Metric, symbol Device:C_Small
- removed D4: 6.8V, Diode_SMD:D_SOD-123, symbol Device:D_Zener_Small_Filled
- removed D5: 1N4148W, Diode_SMD:D_SOD-123, symbol Diode:1N4148W
- removed L2: 3.3uH, Inductor_SMD:L_0603_1608Metric, symbol Device:L_Small
- removed Q2: MMBT3906, Package_TO_SOT_SMD:SOT-23, symbol Transistor_BJT:MMBT3906
- removed R11: 1k, Resistor_SMD:R_0603_1608Metric, symbol Device:R
- removed R2: 200k, Resistor_SMD:R_0603_1608Metric, symbol Device:R_Small
- removed R6: 100k, Resistor_SMD:R_0603_1608Metric, symbol Device:R_Small
- removed R7: 10k, Resistor_SMD:R_0603_1608Metric, symbol Device:R_Small
- removed U1: MT1470, Package_TO_SOT_SMD:SOT-23-6, symbol pslab-mini:MT1470
- added C46, C49: 100uF, Capacitor_SMD:C_0603_1608Metric, symbol Device:C
- added C47: 1.5nF, Capacitor_SMD:C_0603_1608Metric, symbol Device:C
- added C48: 1000uF, Capacitor_SMD:C_0603_1608Metric, symbol Device:C
- added D13: 1N5819WS, Diode_SMD:D_SOD-323, symbol Diode:1N5819WS
- added D14: 6.8V, Diode_SMD:D_SOD-123, symbol Device:D_Zener_Small_Filled
- added D15: 1N4148W, Diode_SMD:D_SOD-123, symbol Diode:1N4148W
- added L6: 88uH, Inductor_SMD:L_0603_1608Metric, symbol Device:L_Small
- added L7: 1uH, Inductor_SMD:L_0603_1608Metric, symbol Device:L_Small
- added Q3: MMBT3906, Package_TO_SOT_SMD:SOT-23, symbol Transistor_BJT:MMBT3906
- added R40: 0.24R, Resistor_SMD:R_0603_1608Metric, symbol Device:R
- added R41, R43: 1k, Resistor_SMD:R_0603_1608Metric, symbol Device:R
- added R42: 6.2k, Resistor_SMD:R_0603_1608Metric, symbol Device:R
- added U12: MC34063ADR, Package_SO:SOIC-8_3.9x4.9mm_P1.27mm, symbol pslab-mini:MC34063ADR
Connections:
- net +5V: now also C46.1, R40.2, U12.6 (Vin)
- net -6V: now also Q3.2 (E)
- net -9V: now also C49.1, L7.1, Q3.3 (C), R43.2
- net GND: now also C46.2, C48.2, C49.2, D14.1 (K), L6.2, R42.1
- new net: R41.1, R42.2, U12.5 (Vfb)
- new net: D15.1 (K), Q3.1 (B), R43.1
- new net: D13.1 (K), L6.1, U12.2 (SwE)
- new net: C47.2, C48.1, D13.2 (A), L7.2, R41.2, U12.4 (GND)
- new net: R40.1, U12.1 (SwC), U12.7 (Ipk), U12.8 (DC)
- new net: C47.1, U12.3 (TC)
- new net: D14.2 (A), D15.2 (A)
Other:
- note added: "Vout = -1.25(1 + 6.2k/1k) = -9V"
- note removed: "Vout=0.8*110k/10k=8.8V"
