File: schematic/pslab-mini.kicad_sch (KiCad schematic)
At the start: 145 parts, among them J2 BAT, J3 Conn_Coaxial, J4 Conn_Coaxial, J5 Conn_02x16_Odd_Even, J6 Conn_01x15_Socket, J7 Conn_02x03_Top_Bottom, J8 USB_C_Receptacle_USB2.0_16P, Q1 MMBT3904, Q2 MMBT3906, SW1 Reset, SW2 Power, U1 MT2496, U10 TL082, U11 ESP32-C3, U12 IP5189T, U2 AP3015A, U4 SP0503BAHT, U5 AMS1117-3.3, U6 STM32H563RIT6, U7 TL082, U8 MCP6S21, U9 MCP6S21, X1 32kHz768, Y1 Crystal_25MHz, Y2 Crystal_40Mhz

Commit message: pcb
Parts:
- removed C45: 1.2pF, Capacitor_SMD:C_0603_1608Metric, symbol Device:C
- added L6: 2.7nH, Inductor_SMD:L_0402_1005Metric, symbol Device:L
- C44: value 1.2pF -> 1pF; footprint Capacitor_SMD:C_0603_1608Metric -> Capacitor_SMD:C_0402_1005Metric
- L5: value 2.4nH -> 3.9nH
- PCB_ANT1: footprint Diode_SMD:D_1206_3216Metric -> RF_Antenna:Johanson_2450AT18x100; Mfr Number RFECA3216060A1T -> 2450AT18A100E; Part Number (LCSC) C127620 -> C89334
- R35, R37, R38, R39: footprint Resistor_SMD:R_0603_1608Metric -> Resistor_SMD:R_0402_1005Metric; Mfr Number RC0603JR-070RL -> RC0402FR-070RL; Part Number (LCSC) C95177 -> C106231
Connections:
- net AGND: now also L6.2; no longer C44.2, PCB_ANT1.2, Y1.2, Y1.4
- net LNA_IN: no longer L5.2
- new net: C44.2, L5.2, L6.1
- new net: Y1.2, Y1.4
- no-connect marks 23 -> 24
Other:
- moved on the sheet: C44
